Commit message: Implementaçao static_transformation_publisher, bem como refatoraçao setup e servo Laser Scan.

File: src/autovehicle_description/urdf/autovehicle.urdf (robot description, URDF)
Before this commit: robot autovehicle, 11 links, 10 joints
Links:
- link base_link: geometry collision mesh filename=package://autovehicle_description/meshes/ford_escape_no_whe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 scale=0.11 0.11 0.11; visual mesh filename=package://autovehicle_description/meshes/ford_escape_no_whe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 scale=0.11 0.11 0.11
- link front_sonar_link: geometry collision box size=${front_sonar_size} ${front_sonar_size} ${front_sonar_size}; visual mesh filename=package://autovehicle_description/meshes/SickLMS.dae scale=0.14 0.14 0.14
- link laser_scan_link: geometry collision box size=0.025 0.025 0.025; visual mesh filename=package://autovehicle_description/meshes/SickLMS.dae scale=0.14 0.14 0.14
- link pantilt_link: geometry collision box size=0.025 0.04 0.025; visual box size=0.025 0.025 0.025
Joints:
- joint pantilt_joint: limit lower=-3.14 upper=3.14 effort=10000 velocity=1000 -> lower=0 upper=0 effort=1.0 velocity=1.0

Commit message: Correçao erro execuçao SLAM.

File: src/autovehicle_description/urdf/autovehicle.urdf (robot description, URDF)
Before this commit: robot autovehicle, 11 links, 10 joints
Links:
- link main_mass: mass ${base_mass} -> None
- link pantilt_link: geometry collision box size=0.025 0.025 0.025; visual box size=0.025 0.025 0.025
Joints:
- joint pantilt_joint: origin xyz=0 0 0.16 rpy=0 0 0 -> xyz=0 0 0.16 rpy=0 0 -1.57

Commit message: Iniciando fase de testes.

File: src/autovehicle_description/urdf/autovehicle.urdf (robot description, URDF)
Before this commit: robot autovehicle, 11 links, 10 joints
Joints:
- joint pantilt_joint: limit lower=0 upper=0 effort=1.0 velocity=1.0 -> lower=-1.57 upper=1.57 effort=1.0 velocity=1.0
